File: EDU_CAR_circuit/wroom-car/wroom-car.kicad_pcb (KiCad board)
At the start: 2 copper layers, 66 x 50 mm, 19 parts, among them M1 Screw_Terminal_01x02, M2 Screw_Terminal_01x02, P1 Conn_01x16_Male, Q1 2N7002, Q2 2N7002, U1 TB6612FNG

Commit message: Upload files New
빠진 부품 수정함
Routing:
- net TRIG: track 0.00 -> 30.5 mm, vias 0 -> 1
- net ECHO: track 0.20 -> 30.3 mm
- added copper zone on B.Cu, net GND
- added copper zone on F.Cu, net GND
Other:
- board text added: "KiMSON"
