File: EDU_CAR_circuit/wroom-car/wroom-car.sch (KiCad schematic (older format))
At the start: 15 parts, among them M1 Screw_Terminal_01x02, M2 Screw_Terminal_01x02, P1 Conn_01x16_Male, Q1 2N7002, Q2 2N7002, U1 TB6612FNG

Commit message: Upload files New
빠진 부품 수정함
Parts:
- added R?: 10K, Resistor_SMD:R_0805_2012Metric, symbol Device:R_US
- added S? (x2): Conn_01x03_Male, Connector_PinHeader_2.54mm:PinHeader_1x03_P2.54mm_Vertical, symbol Connector:Conn_01x03_Male
Connections:
- net +5V: now also R?.1, S?.3 (Pin_3), S?.3 (Pin_3)
- net APWM: now also U1.23 (PWMA)
- net BPWM: now also U1.15 (PWMB)
- net GND: now also U1.10 (PGND2), U1.18 (GND), U1.3 (PGND1), U1.4 (PGND1), U1.9 (PGND2), S?.2 (Pin_2), S?.2 (Pin_2)
- net LEFT: now also S?.1 (Pin_1)
- net RIGHT: now also S?.1 (Pin_1)
- net at U1.1 (AO1), U1.2 (AO1): now also M1.1 (Pin_1)
- net at U1.19 (STBY): now also R?.2
- net at U1.5 (AO2), U1.6 (AO2): now also M1.2 (Pin_2)
Changed lines of the file:
@@
 $EndComp
 Wire Wire Line
-	5150 4950 5850 4950
+	5150 4950 5350 4950
 Wire Wire Line
 	5150 4750 6050 4750
 Wire Wire Line
-	5850 4950 5850 4650
-Wire Wire Line
-	5850 4650 6050 4650
+	5350 4950 5350 4650
+Wire Wire Line
+	5350 4650 6050 4650
 $Comp
 L power:+5V #PWR09
@@
 	1    0    0    -1
 $EndComp
+Text GLabel 3750 4450 0    50   Input ~ 0
+APWM
+Text GLabel 3750 4600 0    50   Input ~ 0
+BPWM
+Wire Wire Line
+	3750 4450 3950 4450
+Wire Wire Line
+	3750 4600 3950 4600
+Wire Wire Line
+	3950 4600 3950 4550
+$Comp
+L Device:R_US R?
+U 1 1 6158AFF1
+P 3550 3900
+F 0 "R?" H 3618 3946 79  0000 L CNN
+F 1 "10K" H 3618 3855 50  0000 L CNN
+F 2 "Resistor_SMD:R_0805_2012Metric" V 3590 3890 50  0001 C CNN
+F 3 "~" H 3550 3900 50  0001 C CNN
+F 4 "C17414" H 3550 3900 50  0001 C CNN "LCSC"
+	1    3550 3900
+	1    0    0    -1
+$EndComp
+$Comp
+L power:+5V #PWR?
+U 1 1 6158B4A1
+P 3550 3650
+F 0 "#PWR?" H 3550 3500 50  0001 C CNN
+F 1 "+5V" H 3565 3823 50  0000 C CNN
+F 2 "" H 3550 3650 50  0001 C CNN
+F 3 "" H 3550 3650 50  0001 C CNN
+	1    3550 3650
+	1    0    0    -1
+$EndComp
+Wire Wire Line
+	3550 3750 3550 3650
+Wire Wire Line
+	3550 4050 3550 4250
+Wire Wire Line
+	3550 4250 3950 4250
+$Comp
+L power:GND #PWR?
+U 1 1 6178C9B0
+P 4250 5800
+F 0 "#PWR?" H 4250 5550 50  0001 C CNN
+F 1 "GND" H 4255 5627 50  0000 C CNN
+F 2 "" H 4250 5800 50  0001 C CNN
+F 3 "" H 4250 5800 50  0001 C CNN
+	1    4250 5800
+	1    0    0    -1
+$EndComp
+Wire Wire Line
+	4250 5650 4250 5750
+Wire Wire Line
+	4850 5650 4850 5750
+Wire Wire Line
+	4850 5750 4650 5750
+Connection ~ 4250 5750
+Wire Wire Line
+	4250 5750 4250 5800
+Wire Wire Line
+	4650 5650 4650 5750
+Connection ~ 4650 5750
+Wire Wire Line
+	4650 5750 4250 5750
+$Comp
+L Connector:Conn_01x03_Male S?
+U 1 1 61793DBF
+P 7400 2300
+F 0 "S?" H 7508 2581 50  0000 C CNN
+F 1 "Conn_01x03_Male" H 7508 2490 50  0000 C CNN
+F 2 "Connector_PinHeader_2.54mm:PinHeader_1x03_P2.54mm_Vertical" H 7400 2300 50  0001 C CNN
+F 3 "~" H 7400 2300 50  0001 C CNN
+	1    7400 2300
+	1    0    0    -1
+$EndComp
+$Comp
+L Connector:Conn_01x03_Male S?
+U 1 1 6179532A
+P 9050 2300
+F 0 "S?" H 9158 2581 50  0000 C CNN
+F 1 "Conn_01x03_Male" H 9158 2490 50  0000 C CNN
+F 2 "Connector_PinHeader_2.54mm:PinHeader_1x03_P2.54mm_Vertical" H 9050 2300 50  0001 C CNN
+F 3 "~" H 9050 2300 50  0001 C CNN
+	1    9050 2300
+	1    0    0    -1
+$EndComp
+Text GLabel 8000 2200 2    55   Input ~ 0
+LEFT
+Text GLabel 9700 2200 2    55   Input ~ 0
+RIGHT
+$Comp
+L power:GND #PWR?
+U 1 1 6179E485
+P 7800 2550
+F 0 "#PWR?" H 7800 2300 50  0001 C CNN
+F 1 "GND" H 7805 2377 50  0000 C CNN
+F 2 "" H 7800 2550 50  0001 C CNN
+F 3 "" H 7800 2550 50  0001 C CNN
+	1    7800 2550
+	1    0    0    -1
+$EndComp
+$Comp
+L power:GND #PWR?
+U 1 1 6179E946
+P 9450 2550
+F 0 "#PWR?" H 9450 2300 50  0001 C CNN
+F 1 "GND" H 9455 2377 50  0000 C CNN
+F 2 "" H 9450 2550 50  0001 C CNN
+F 3 "" H 9450 2550 50  0001 C CNN
+	1    9450 2550
+	1    0    0    -1
+$EndComp
+$Comp
+L power:+5V #PWR?
+U 1 1 6179EC64
+P 7850 1950
+F 0 "#PWR?" H 7850 1800 50  0001 C CNN
+F 1 "+5V" H 7865 2123 50  0000 C CNN
+F 2 "" H 7850 1950 50  0001 C CNN
+F 3 "" H 7850 1950 50  0001 C CNN
+	1    7850 1950
+	1    0    0    -1
+$EndComp
+$Comp
+L power:+5V #PWR?
+U 1 1 6179F239
+P 9500 1950
+F 0 "#PWR?" H 9500 1800 50  0001 C CNN
+F 1 "+5V" H 9515 2123 50  0000 C CNN
+F 2 "" H 9500 1950 50  0001 C CNN
+F 3 "" H 9500 1950 50  0001 C CNN
+	1    9500 1950
+	1    0    0    -1
+$EndComp
+Wire Wire Line
+	7600 2200 8000 2200
+Wire Wire Line
+	7850 1950 7850 2400
+Wire Wire Line
+	7850 2400 7600 2400
+Wire Wire Line
+	9500 1950 9500 2400
+Wire Wire Line
+	9500 2400 9250 2400
+Wire Wire Line
+	9250 2200 9700 2200
+Wire Wire Line
+	9250 2300 9450 2300
+Wire Wire Line
+	9450 2300 9450 2550
+Wire Wire Line
+	7600 2300 7800 2300
+Wire Wire Line
+	7800 2300 7800 2550
+Wire Wire Line
+	6050 4450 5150 4450
+Wire Wire Line
+	6050 4350 5350 4350
+Wire Wire Line
+	5350 4350 5350 4250
+Wire Wire Line
+	5350 4250 5150 4250
 $EndSCHEMATC

Commit message: Add files via upload
Parts:
- gave numbers to parts that had none: 3
Changed lines of the file:
@@
 	3950 4600 3950 4550
 $Comp
-L Device:R_US R?
+L Device:R_US R5
 U 1 1 6158AFF1
 P 3550 3900
-F 0 "R?" H 3618 3946 79  0000 L CNN
+F 0 "R5" H 3618 3946 79  0000 L CNN
 F 1 "10K" H 3618 3855 50  0000 L CNN
 F 2 "Resistor_SMD:R_0805_2012Metric" V 3590 3890 50  0001 C CNN
@@
 $EndComp
 $Comp
-L power:+5V #PWR?
+L power:+5V #PWR0101
 U 1 1 6158B4A1
 P 3550 3650
-F 0 "#PWR?" H 3550 3500 50  0001 C CNN
+F 0 "#PWR0101" H 3550 3500 50  0001 C CNN
 F 1 "+5V" H 3565 3823 50  0000 C CNN
 F 2 "" H 3550 3650 50  0001 C CNN
@@
 	3550 4250 3950 4250
 $Comp
-L power:GND #PWR?
+L power:GND #PWR0102
 U 1 1 6178C9B0
 P 4250 5800
-F 0 "#PWR?" H 4250 5550 50  0001 C CNN
+F 0 "#PWR0102" H 4250 5550 50  0001 C CNN
 F 1 "GND" H 4255 5627 50  0000 C CNN
 F 2 "" H 4250 5800 50  0001 C CNN
@@
 	4650 5750 4250 5750
 $Comp
-L Connector:Conn_01x03_Male S?
+L Connector:Conn_01x03_Male S1
 U 1 1 61793DBF
 P 7400 2300
-F 0 "S?" H 7508 2581 50  0000 C CNN
+F 0 "S1" H 7508 2581 50  0000 C CNN
 F 1 "Conn_01x03_Male" H 7508 2490 50  0000 C CNN
 F 2 "Connector_PinHeader_2.54mm:PinHeader_1x03_P2.54mm_Vertical" H 7400 2300 50  0001 C CNN
@@
 $EndComp
 $Comp
-L Connector:Conn_01x03_Male S?
+L Connector:Conn_01x03_Male S2
 U 1 1 6179532A
 P 9050 2300
-F 0 "S?" H 9158 2581 50  0000 C CNN
+F 0 "S2" H 9158 2581 50  0000 C CNN
 F 1 "Conn_01x03_Male" H 9158 2490 50  0000 C CNN
 F 2 "Connector_PinHeader_2.54mm:PinHeader_1x03_P2.54mm_Vertical" H 9050 2300 50  0001 C CNN
@@
 RIGHT
 $Comp
-L power:GND #PWR?
+L power:GND #PWR0103
 U 1 1 6179E485
 P 7800 2550
-F 0 "#PWR?" H 7800 2300 50  0001 C CNN
+F 0 "#PWR0103" H 7800 2300 50  0001 C CNN
 F 1 "GND" H 7805 2377 50  0000 C CNN
 F 2 "" H 7800 2550 50  0001 C CNN
@@
 $EndComp
 $Comp
-L power:GND #PWR?
+L power:GND #PWR0104
 U 1 1 6179E946
 P 9450 2550
-F 0 "#PWR?" H 9450 2300 50  0001 C CNN
+F 0 "#PWR0104" H 9450 2300 50  0001 C CNN
 F 1 "GND" H 9455 2377 50  0000 C CNN
 F 2 "" H 9450 2550 50  0001 C CNN
@@
 $EndComp
 $Comp
-L power:+5V #PWR?
+L power:+5V #PWR0105
 U 1 1 6179EC64
 P 7850 1950
-F 0 "#PWR?" H 7850 1800 50  0001 C CNN
+F 0 "#PWR0105" H 7850 1800 50  0001 C CNN
 F 1 "+5V" H 7865 2123 50  0000 C CNN
 F 2 "" H 7850 1950 50  0001 C CNN
@@
 $EndComp
 $Comp
-L power:+5V #PWR?
+L power:+5V #PWR0106
 U 1 1 6179F239
 P 9500 1950
-F 0 "#PWR?" H 9500 1800 50  0001 C CNN
+F 0 "#PWR0106" H 9500 1800 50  0001 C CNN
 F 1 "+5V" H 9515 2123 50  0000 C CNN
 F 2 "" H 9500 1950 50  0001 C CNN
